Commit message: removed battery pack weight

File: urdf/atlas_v5_reflex_hands.urdf (robot description, URDF)
Before this commit: robot atlas, 71 links, 70 joints
Links:
- added link l_end_eff
- added link r_end_eff
- link utorso: mass 84.409 -> 62.563
Joints:
- added joint l_robotiq_end_eff_virtual_joint: type fixed, parent l_palm, child l_end_eff, origin xyz=0.0 0.0 0.15 rpy=0 -1.57079633 0
- added joint r_robotiq_end_eff_virtual_joint: type fixed, parent r_palm, child r_end_eff, origin xyz=0.0 0.0 0.15 rpy=0 -1.57079633 0
- joint l_fixed: child l_fixed_dummy -> l_palm; origin xyz=0 0 0 rpy=0 0 0 -> xyz=-0.00125 -0.15 0.0 rpy=0 1.57295 -1.57295
- joint l_fixed_dummy: child l_fixed_dummy2 -> l_fixed_dummy; parent l_fixed_dummy -> l_palm
- joint l_fixed_dummy2: child l_palm -> l_fixed_dummy2; origin xyz=-0.00125 -0.15 0.0 rpy=0 1.57295 -1.57295 -> xyz=0 0 0 rpy=0 0 0; parent l_fixed_dummy2 -> l_fixed_dummy
- joint r_fixed: child r_fixed_dummy -> r_palm; origin xyz=0 0 0 rpy=0 0 0 -> xyz=-0.00125 -0.15 0.0 rpy=1.57295 1.57295 0
- joint r_fixed_dummy: child r_fixed_dummy2 -> r_fixed_dummy; parent r_fixed_dummy -> r_palm
- joint r_fixed_dummy2: child r_palm -> r_fixed_dummy2; origin xyz=-0.00125 -0.15 0.0 rpy=1.57295 1.57295 0 -> xyz=0 0 0 rpy=0 0 0; parent r_fixed_dummy2 -> r_fixed_dummy

Commit message: Added collision to fingers

File: urdf/atlas_v5_reflex_hands.urdf (robot description, URDF)
Before this commit: robot atlas, 73 links, 72 joints
Links:
- link l_finger_1_1: geometry collision mesh filename=package://reflex_hand_model/meshes/swivel_1.STL; visual mesh filename=package://reflex_hand_model/meshes/swivel_1.STL
- link l_finger_1_2: geometry collision mesh filename=package://reflex_hand_model/meshes/proximal_1.STL; visual mesh filename=package://reflex_hand_model/meshes/proximal_1.STL
- link l_finger_1_3: geometry collision mesh filename=package://reflex_hand_model/meshes/distal_1.STL; visual mesh filename=package://reflex_hand_model/meshes/distal_1.STL
- link l_finger_2_1: geometry collision mesh filename=package://reflex_hand_model/meshes/swivel_1.STL; visual mesh filename=package://reflex_hand_model/meshes/swivel_1.STL
- link l_finger_2_2: geometry collision mesh filename=package://reflex_hand_model/meshes/proximal_1.STL; visual mesh filename=package://reflex_hand_model/meshes/proximal_1.STL
- link l_finger_2_3: geometry collision mesh filename=package://reflex_hand_model/meshes/distal_1.STL; visual mesh filename=package://reflex_hand_model/meshes/distal_1.STL
- link l_finger_3_1: geometry collision mesh filename=package://reflex_hand_model/meshes/swivel_1.STL; visual mesh filename=package://reflex_hand_model/meshes/swivel_1.STL
- link l_finger_3_2: geometry collision mesh filename=package://reflex_hand_model/meshes/proximal_1.STL; visual mesh filename=package://reflex_hand_model/meshes/proximal_1.STL
- link l_finger_3_3: geometry collision mesh filename=package://reflex_hand_model/meshes/distal_1.STL; visual mesh filename=package://reflex_hand_model/meshes/distal_1.STL
- link r_finger_1_1: geometry collision mesh filename=package://reflex_hand_model/meshes/swivel_1.STL; visual mesh filename=package://reflex_hand_model/meshes/swivel_1.STL
- link r_finger_1_2: geometry collision mesh filename=package://reflex_hand_model/meshes/proximal_1.STL; visual mesh filename=package://reflex_hand_model/meshes/proximal_1.STL
- link r_finger_1_3: geometry collision mesh filename=package://reflex_hand_model/meshes/distal_1.STL; visual mesh filename=package://reflex_hand_model/meshes/distal_1.STL
- link r_finger_2_1: geometry collision mesh filename=package://reflex_hand_model/meshes/swivel_1.STL; visual mesh filename=package://reflex_hand_model/meshes/swivel_1.STL
- link r_finger_2_2: geometry collision mesh filename=package://reflex_hand_model/meshes/proximal_1.STL; visual mesh filename=package://reflex_hand_model/meshes/proximal_1.STL
- link r_finger_2_3: geometry collision mesh filename=package://reflex_hand_model/meshes/distal_1.STL; visual mesh filename=package://reflex_hand_model/meshes/distal_1.STL
- link r_finger_3_1: geometry collision mesh filename=package://reflex_hand_model/meshes/swivel_1.STL; visual mesh filename=package://reflex_hand_model/meshes/swivel_1.STL
- link r_finger_3_2: geometry collision mesh filename=package://reflex_hand_model/meshes/proximal_1.STL; visual mesh filename=package://reflex_hand_model/meshes/proximal_1.STL
- link r_finger_3_3: geometry collision mesh filename=package://reflex_hand_model/meshes/distal_1.STL; visual mesh filename=package://reflex_hand_model/meshes/distal_1.STL
